Commit message: Joint state publisher GUI
Got the joint state publisher gui to work and fixed prior xacro issues with script

File: urdf/robot_definition.urdf (robot description, URDF)
Before this commit: robot navvis, 6 links, 5 joints
Links:
- added link wheel_center; collision cylinder length=0.05 radius=0.15; visual cylinder length=0.05 radius=0.15
- added link wheel_right; collision cylinder length=0.05 radius=0.2; visual cylinder length=0.05 radius=0.2
Joints:
- added joint base_wheel_center_joint: type fixed, parent base, child wheel_center, origin xyz=0.1 0.0 0.0 rpy=-1.57 0.0 0.0
- added joint base_wheel_right_joint: type fixed, parent base, child wheel_right, origin xyz=-0.1 -0.4 0.0 rpy=-1.5707963267948966 0.0 0.0
- joint wheel_left_joint: origin xyz=-0.1 0.4 0.0 rpy=-1.57 0.0 0.0 -> xyz=-0.1 0.4 0.0 rpy=-1.5707963267948966 0.0 0.0

File: urdf/robot_definition.xacro (robot description, xacro)
@@ -64,6 +64,20 @@
 		</collision>
 	</link>
+	<link name="wheel_center">
+		<visual>
+			<origin xyz="0.0 0.0 0.0" rpy="0.0 0.0 0.0" />
+			<geometry>
+				<cylinder radius="0.15" length = '0.05'/>
+			</geometry>
+		</visual>
+		<collision>
+			<origin xyz="0.0 0.0 0.0" rpy="0.0 0.0 0.0" />
+			<geometry>
+				<cylinder radius="0.15" length = '0.05'/>
+			</geometry>
+		</collision>
+	</link>
 	<xacro:macro name="xacro_name" params="side reflect">
-		<link name="wheel_left">
+		<link name="wheel_${side}">
 			<visual>
 				<geometry>
@@ -77,4 +91,11 @@
 			</collision>
 		</link>
+		<joint name = 'base_wheel_${side}_joint' type ="continuous">
+			<parent link = 'base'/>
+			<child link='wheel_${side}'/>
+			<origin xyz="-0.1 ${reflect*0.4} 0.0" rpy="-${pi/2} 0.0 0.0"/>
+			<axis xyz = '0 0 1'/>
+			<limit effort='30' velocity='5'/>
+		</joint>
 	</xacro:macro>
 	<joint name = 'base_laser_vert_bottom_joint' type = "fixed">
@@ -98,11 +119,11 @@
 		<origin xyz="0.2325 0.0001 1.9201" rpy="0.0012 0.1146 -0.0015"/>
 	</joint>
-	<xacro:macro name="xacro_name" params="side reflect">
-		<joint name = 'wheel_left_joint' type = "fixed">
-			<parent link = 'base'/>
-			<child link='wheel_left'/>
-			<origin xyz="-0.1 0.4 0.0" rpy="-1.57 0.0 0.0"/>
-		</joint>
-	</xacro:macro>
+	<joint name = 'base_wheel_center_joint' type = "continuous">
+		<parent link = 'base'/>
+		<child link='wheel_center'/>
+		<origin xyz="0.1 0.0 -0.05" rpy="-1.57 0.0 0.0"/>
+		<axis xyz = '0 0 1'/>
+		<limit effort='30' velocity='5'/>
+	</joint>
 	<xacro:xacro_name side="left" reflect="1" />
 	<xacro:xacro_name side="right" reflect="-1" />

File: urdf/urdf_from_xacro.urdf (robot description, URDF)
Before this commit: robot navvis, 5 links, 5 joints
Links:
- added link wheel_left; collision cylinder length=0.05 radius=0.2; visual cylinder length=0.05 radius=0.2
- added link wheel_right; collision cylinder length=0.05 radius=0.2; visual cylinder length=0.05 radius=0.2
Joints:
- added joint wheel_right_joint: type fixed, parent base, child wheel_right, origin xyz=-0.1 -0.4 0.0 rpy=-1.5707963267948966 0.0 0.0
- joint wheel_left_joint: origin xyz=-0.1 0.4 0.0 rpy=-1.57 0.0 0.0 -> xyz=-0.1 0.4 0.0 rpy=-1.5707963267948966 0.0 0.0
